Commit message: modified:   README.md 	renamed:    d435i_depth/__init__.py -> d455_depth/__init__.py 	modified:   launch/depth.launch.py 	deleted:    meshes/d435.dae 	new file:   meshes/d455.stl 	modified:   package.xml 	renamed:    resource/d435i_depth -> resource/d455_depth 	modified:   setup.cfg 	modified:   setup.py 	deleted:    urdf/d435.urdf.xacro 	deleted:    urdf/d435i.gazebo.xacro 	deleted:    urdf/d435i.urdf.xacro 	deleted:    urdf/d435i_imu_modules.urdf.xacro 	new file:   urdf/d455.urdf.xacro 	deleted:    urdf/test_d435i.urdf.xacro 	new file:   urdf/test_d455_camera.urdf.xacro 	modified:   urdf/usb_plug.urdf.xacro

File: urdf/usb_plug.urdf.xacro (robot description, xacro)
@@ -33,5 +33,5 @@
         <geometry>
           <!--box size="0.044850 0.008 0.0185" /-->
-          <mesh filename="file:///$(find d435i_depth)/meshes/plug.stl" />
+          <mesh filename="file:///$(find d455_depth)/meshes/plug.stl" />
         </geometry>
         <material name="plastic"/>
@@ -41,5 +41,5 @@
         <geometry>
           <!--box size="0.044850 0.008 0.0185" /-->
-          <mesh filename="file:///$(find d435i_depth)/meshes/plug_collision.stl" />
+          <mesh filename="file:///$(find d455_depth)/meshes/plug_collision.stl" />
         </geometry>
       </collision>
