Commit message: modified:   README.md 	modified:   launch/depth.launch.py 	modified:   package.xml 	renamed:    d435i_depth/__init__.py -> realsense_cam/__init__.py 	renamed:    resource/d435i_depth -> resource/realsense_cam 	modified:   setup.cfg 	modified:   setup.py 	modified:   urdf/d435.urdf.xacro 	modified:   urdf/d435i.urdf.xacro 	modified:   urdf/test_d435i.urdf.xacro 	modified:   urdf/usb_plug.urdf.xacro

File: urdf/d435.urdf.xacro (robot description, xacro)
@@ -21,6 +21,6 @@
 <robot name="sensor_d435" xmlns:xacro="http://ros.org/wiki/xacro">
   <!-- Includes -->
-  <xacro:include filename="$(find d435i_depth)/urdf/materials.urdf.xacro" />
-  <xacro:include filename="$(find d435i_depth)/urdf/usb_plug.urdf.xacro" />
+  <xacro:include filename="$(find realsense_cam)/urdf/materials.urdf.xacro" />
+  <xacro:include filename="$(find realsense_cam)/urdf/usb_plug.urdf.xacro" />
   <xacro:macro name="sensor_d435" params="parent *origin name:=camera use_nominal_extrinsics:=false add_plug:=false use_mesh:=true">
     <xacro:property name="M_PI" value="3.1415926535897931" />
@@ -66,5 +66,5 @@
           <origin xyz="${d435_zero_depth_to_glass + d435_glass_to_front} ${-d435_cam_depth_py} 0" rpy="${M_PI/2} 0 ${M_PI/2}"/>
           <geometry>
-            <mesh filename="file:///$(find d435i_depth)/meshes/d435.dae" />
+            <mesh filename="file:///$(find realsense_cam)/meshes/d435.dae" />
           </geometry>
         </xacro:if>

File: urdf/d435i.urdf.xacro (robot description, xacro)
@@ -20,6 +20,6 @@
 -->
 <robot name="sensor_d435i" xmlns:xacro="http://ros.org/wiki/xacro">
-  <xacro:include filename="$(find d435i_depth)/urdf/d435.urdf.xacro"/>
-  <xacro:include filename="$(find d435i_depth)/urdf/d435i_imu_modules.urdf.xacro"/>
+  <xacro:include filename="$(find realsense_cam)/urdf/d435.urdf.xacro"/>
+  <xacro:include filename="$(find realsense_cam)/urdf/d435i_imu_modules.urdf.xacro"/>
   <xacro:macro name="sensor_d435i" params="parent *origin name:=camera use_nominal_extrinsics:=false">
     <xacro:sensor_d435 parent="${parent}" name="${name}" use_nominal_extrinsics="${use_nominal_extrinsics}">
@@ -28,4 +28,4 @@
     <xacro:d435i_imu_modules name="${name}" use_nominal_extrinsics="${use_nominal_extrinsics}"/>
   </xacro:macro>
-  <xacro:include filename="$(find d435i_depth)/urdf/d435i.gazebo.xacro"/>
+  <xacro:include filename="$(find realsense_cam)/urdf/d435i.gazebo.xacro"/>
 </robot>

File: urdf/test_d435i.urdf.xacro (robot description, xacro)
@@ -2,5 +2,5 @@
 <robot name="realsense2_camera" xmlns:xacro="http://www.ros.org/wiki/xacro">
   <xacro:arg name="use_nominal_extrinsics" default="true" />
-  <xacro:include filename="$(find d435i_depth)/urdf/d435i.urdf.xacro"/>
+  <xacro:include filename="$(find realsense_cam)/urdf/d435i.urdf.xacro"/>
   <link name="base_screw"/>
   <xacro:sensor_d435i parent="base_screw" use_nominal_extrinsics="$(arg use_nominal_extrinsics)">

File: urdf/usb_plug.urdf.xacro (robot description, xacro)
@@ -33,5 +33,5 @@
         <geometry>
           <!--box size="0.044850 0.008 0.0185" /-->
-          <mesh filename="file:///$(find d435i_depth)/meshes/plug.stl" />
+          <mesh filename="file:///$(find realsense_cam)/meshes/plug.stl" />
         </geometry>
         <material name="plastic"/>
@@ -41,5 +41,5 @@
         <geometry>
           <!--box size="0.044850 0.008 0.0185" /-->
-          <mesh filename="file:///$(find d435i_depth)/meshes/plug_collision.stl" />
+          <mesh filename="file:///$(find realsense_cam)/meshes/plug_collision.stl" />
         </geometry>
       </collision>
