Commit message: modified:   urdf/test_d455_camera.urdf.xacro

File: urdf/test_d455_camera.urdf.xacro (robot description, xacro)
@@ -3,6 +3,6 @@
   <xacro:arg name="use_nominal_extrinsics" default="true"/>
   <xacro:include filename="$(find realsense_cam)/urdf/d455.urdf.xacro" />
-  <link name="base_link" />
-  <xacro:sensor_d455 parent="base_link" use_nominal_extrinsics="$(arg use_nominal_extrinsics)">
+  <link name="base_screw" />
+  <xacro:sensor_d455 parent="base_screw" use_nominal_extrinsics="$(arg use_nominal_extrinsics)">
     <origin xyz="0 0 0" rpy="0 0 0"/>
   </xacro:sensor_d455>
