Commit message: modified:   README.md 	modified:   launch/depth.launch.py 	modified:   package.xml 	renamed:    d455_depth/__init__.py -> realsense_cam/__init__.py 	renamed:    resource/d455_depth -> resource/realsense_cam 	modified:   setup.cfg 	modified:   setup.py 	modified:   urdf/d455.urdf.xacro 	modified:   urdf/test_d455_camera.urdf.xacro 	modified:   urdf/usb_plug.urdf.xacro

File: urdf/d455.urdf.xacro (robot description, xacro)
@@ -8,6 +8,6 @@
 <robot name="sensor_d455" xmlns:xacro="http://ros.org/wiki/xacro">
   <!-- Includes -->
-  <xacro:include filename="$(find d455_depth)/urdf/materials.urdf.xacro" />
-  <xacro:include filename="$(find d455_depth)/urdf/usb_plug.urdf.xacro" />
+  <xacro:include filename="$(find realsense_cam)/urdf/materials.urdf.xacro" />
+  <xacro:include filename="$(find realsense_cam)/urdf/usb_plug.urdf.xacro" />
   <xacro:macro name="sensor_d455" params="parent *origin name:=camera use_nominal_extrinsics:=false">
     <xacro:arg name="add_plug" default="false" />
@@ -55,5 +55,5 @@
         <geometry>
           <!-- <box size="${d455_cam_depth} ${d455_cam_width} ${d455_cam_height}"/> -->
-	        <mesh filename="file:///$(find d455_depth)/meshes/d455.stl" scale="0.001 0.001 0.001" />
+	        <mesh filename="file:///$(find realsense_cam)/meshes/d455.stl" scale="0.001 0.001 0.001" />
         </geometry>
         <material name="aluminum"/>

File: urdf/test_d455_camera.urdf.xacro (robot description, xacro)
@@ -2,5 +2,5 @@
 <robot name="realsense2_camera" xmlns:xacro="http://ros.org/wiki/xacro">
   <xacro:arg name="use_nominal_extrinsics" default="true"/>
-  <xacro:include filename="$(find d455_depth)/urdf/d455.urdf.xacro" />
+  <xacro:include filename="$(find realsense_cam)/urdf/d455.urdf.xacro" />
   <link name="base_link" />
   <xacro:sensor_d455 parent="base_link" use_nominal_extrinsics="$(arg use_nominal_extrinsics)">

File: urdf/usb_plug.urdf.xacro (robot description, xacro)
@@ -33,5 +33,5 @@
         <geometry>
           <!--box size="0.044850 0.008 0.0185" /-->
-          <mesh filename="file:///$(find d455_depth)/meshes/plug.stl" />
+          <mesh filename="file:///$(find realsense_cam)/meshes/plug.stl" />
         </geometry>
         <material name="plastic"/>
@@ -41,5 +41,5 @@
         <geometry>
           <!--box size="0.044850 0.008 0.0185" /-->
-          <mesh filename="file:///$(find d455_depth)/meshes/plug_collision.stl" />
+          <mesh filename="file:///$(find realsense_cam)/meshes/plug_collision.stl" />
         </geometry>
       </collision>

Commit message: modified:   launch/depth.launch.py 	modified:   urdf/d455.urdf.xacro

File: urdf/d455.urdf.xacro (robot description, xacro)
@@ -10,5 +10,5 @@
   <xacro:include filename="$(find realsense_cam)/urdf/materials.urdf.xacro" />
   <xacro:include filename="$(find realsense_cam)/urdf/usb_plug.urdf.xacro" />
-  <xacro:include filename="$(find realsense_cam)/urdf/d455.gazebo.xacro"/>
+  <!--<xacro:include filename="$(find realsense_cam)/urdf/d455.gazebo.xacro"/>-->
   <xacro:macro name="sensor_d455" params="parent *origin name:=camera use_nominal_extrinsics:=false">
     <xacro:arg name="add_plug" default="false" />
@@ -96,5 +96,5 @@
       <link name="${name}_infra1_frame"/>
       <joint name="${name}_infra1_optical_joint" type="fixed">
-        <origin xyz="0 0 0" rpy="${-M_PI/2} 0 ${-M_PI/2}" />
+        <origin xyz="0 0 0" rpy="0 0 0" />
         <parent link="${name}_infra1_frame" />
         <child link="${name}_infra1_optical_frame" />
@@ -109,5 +109,5 @@
       <link name="${name}_infra2_frame"/>
       <joint name="${name}_infra2_optical_joint" type="fixed">
-        <origin xyz="0 0 0" rpy="${-M_PI/2} 0 ${-M_PI/2}" />
+        <origin xyz="0 0 0" rpy="0 0 0" />
         <parent link="${name}_infra2_frame" />
         <child link="${name}_infra2_optical_frame" />
